Commit message: most things working simulation doesn't show the real thing

File: schunk_description/urdf/sdh/sdh.gazebo.xacro (robot description, xacro)
@@ -6,111 +6,123 @@
 	<xacro:macro name="schunk_sdh_gazebo" params="name">
 		<gazebo reference="${name}_palm_link">
-			<material>Gazebo/Grey</material>
+			<material>Schunk/LightGrey</material>
 			<turnGravityOff>false</turnGravityOff>
 		</gazebo>
 		<gazebo reference="${name}_finger_11_link">
-			<material>Gazebo/Black</material>
+			<material>Schunk/LightGrey</material>
 			<turnGravityOff>false</turnGravityOff>
 		</gazebo>
 		<gazebo reference="${name}_finger_12_link">
 			<selfCollide>true</selfCollide>
-			<sensor:contact name="${name}_finger_12_contact_sensor">
-				<geom>${name}_finger_12_link_geom</geom>
-				<updateRate>100.0</updateRate>
-				<controller:gazebo_ros_bumper name="${name}_finger_12_gazebo_ros_bumper_controller" plugin="libgazebo_ros_bumper.so">
+			<sensor name='${name}_finger_12_contact_sensor' type='contact'>
+				<always_on>true</always_on>
+				<update_rate>100</update_rate>
+				<contact>
+					<collision>${name}_finger_12_link_geom</collision>
+				</contact>
+				<plugin name="${name}_finger_12_gazebo_ros_bumper_controller" filename="libgazebo_ros_bumper.so">
 					<alwaysOn>true</alwaysOn>
 					<updateRate>100.0</updateRate>
 					<frameName>${name}_finger_12_link</frameName>
 					<bumperTopicName>${name}_finger_12_bumper</bumperTopicName>
-					<interface:bumper name="${name}_finger_12_bumper_iface" />
-				</controller:gazebo_ros_bumper>
-			</sensor:contact>
-			<material>IPA/Grey1</material>
+				</plugin>
+			</sensor>
+			<material>Schunk/LightGrey</material>
 			<turnGravityOff>false</turnGravityOff>
 		</gazebo>
 		<gazebo reference="${name}_finger_13_link">
 			<selfCollide>true</selfCollide>
-			<sensor:contact name="${name}_finger_13_contact_sensor">
-				<geom>${name}_finger_13_link_geom</geom>
-				<updateRate>100.0</updateRate>
-				<controller:gazebo_ros_bumper name="${name}_finger_13_gazebo_ros_bumper_controller" plugin="libgazebo_ros_bumper.so">
+			<sensor name='${name}_finger_13_contact_sensor' type='contact'>
+				<always_on>true</always_on>
+				<update_rate>100</update_rate>
+				<contact>
+					<collision>${name}_finger_13_link_geom</collision>
+				</contact>
+				<plugin name="${name}_finger_13_gazebo_ros_bumper_controller" filename="libgazebo_ros_bumper.so">
 					<alwaysOn>true</alwaysOn>
 					<updateRate>100.0</updateRate>
 					<frameName>${name}_finger_13_link</frameName>
 					<bumperTopicName>${name}_finger_13_bumper</bumperTopicName>
-					<interface:bumper name="${name}_finger_13_bumper_iface" />
-				</controller:gazebo_ros_bumper>
-			</sensor:contact>
-			<material>IPA/Grey2</material>
+				</plugin>
+			</sensor>
+			<material>Schunk/LightGrey</material>
 		</gazebo>
 		<gazebo reference="${name}_finger_21_link">
-			<material>Gazebo/Black</material>
+			<material>Schunk/LightGrey</material>
 			<turnGravityOff>false</turnGravityOff>
 		</gazebo>
 		<gazebo reference="${name}_finger_22_link">
-		<selfCollide>true</selfCollide>
-			<sensor:contact name="${name}_finger_22_contact_sensor">
-				<geom>${name}_finger_22_link_geom</geom>
-				<updateRate>100.0</updateRate>
-				<controller:gazebo_ros_bumper name="${name}_finger_22_gazebo_ros_bumper_controller" plugin="libgazebo_ros_bumper.so">
+			<selfCollide>true</selfCollide>
+			<sensor name='${name}_finger_22_contact_sensor' type='contact'>
+				<always_on>true</always_on>
+				<update_rate>100</update_rate>
+				<contact>
+					<collision>${name}_finger_22_link_geom</collision>
+				</contact>
+				<plugin name="${name}_finger_22_gazebo_ros_bumper_controller" filename="libgazebo_ros_bumper.so">
 					<alwaysOn>true</alwaysOn>
 					<updateRate>100.0</updateRate>
 					<frameName>${name}_finger_22_link</frameName>
 					<bumperTopicName>${name}_finger_22_bumper</bumperTopicName>
-					<interface:bumper name="${name}_finger_22_bumper_iface" />
-				</controller:gazebo_ros_bumper>
-			</sensor:contact>
-			<material>IPA/Grey1</material>
+				</plugin>
+			</sensor>
+			<material>Schunk/LightGrey</material>
 			<turnGravityOff>false</turnGravityOff>
 		</gazebo>
 		<gazebo reference="${name}_finger_23_link">
 			<selfCollide>true</selfCollide>
-			<sensor:contact name="${name}_finger_23_contact_sensor">
-				<geom>${name}_finger_23_link_geom</geom>
-				<updateRate>100.0</updateRate>
-				<controller:gazebo_ros_bumper name="${name}_finger_23_gazebo_ros_bumper_controller" plugin="libgazebo_ros_bumper.so">
+			<sensor name='${name}_finger_23_contact_sensor' type='contact'>
+				<always_on>true</always_on>
+				<update_rate>100</update_rate>
+				<contact>
+					<collision>${name}_finger_23_link_geom</collision>
+				</contact>
+				<plugin name="${name}_finger_23_gazebo_ros_bumper_controller" filename="libgazebo_ros_bumper.so">
 					<alwaysOn>true</alwaysOn>
 					<updateRate>100.0</updateRate>
 					<frameName>${name}_finger_23_link</frameName>
 					<bumperTopicName>${name}_finger_23_bumper</bumperTopicName>
-					<interface:bumper name="${name}_finger_23_bumper_iface" />
-				</controller:gazebo_ros_bumper>
-			</sensor:contact>
-			<material>IPA/Grey2</material>
+				</plugin>
+			</sensor>
+			<material>Schunk/LightGrey</material>
 		</gazebo>
 		<gazebo reference="${name}_thumb_1_link">
-			<material>Gazebo/Black</material>
+			<material>Schunk/LightGrey</material>
 			<turnGravityOff>false</turnGravityOff>
 		</gazebo>
 		<gazebo reference="${name}_thumb_2_link">
 			<selfCollide>true</selfCollide>
-			<sensor:contact name="${name}_thumb_2_contact_sensor">
-				<geom>${name}_thumb_2_link_geom</geom>
-				<updateRate>100.0</updateRate>
-				<controller:gazebo_ros_bumper name="${name}_thumb_2_gazebo_ros_bumper_controller" plugin="libgazebo_ros_bumper.so">
+			<sensor name='${name}_thumb_2_contact_sensor' type='contact'>
+				<always_on>true</always_on>
+				<update_rate>100</update_rate>
+				<contact>
+					<collision>${name}_thumb_2_link_geom</collision>
+				</contact>
+				<plugin name="${name}_thumb_2_gazebo_ros_bumper_controller" filename="libgazebo_ros_bumper.so">
 					<alwaysOn>true</alwaysOn>
 					<updateRate>100.0</updateRate>
 					<frameName>${name}_thumb_2_link</frameName>
 					<bumperTopicName>${name}_thumb_2_bumper</bumperTopicName>
-					<interface:bumper name="${name}_thumb_2_bumper_iface" />
-				</controller:gazebo_ros_bumper>
-			</sensor:contact>
-			<material>IPA/Grey1</material>
+				</plugin>
+			</sensor>
+			<material>Schunk/LightGrey</material>
 			<turnGravityOff>false</turnGravityOff>
 		</gazebo>
 		<gazebo reference="${name}_thumb_3_link">
 			<selfCollide>true</selfCollide>
-			<sensor:contact name="${name}_thumb_3_contact_sensor">
-				<geom>${name}_thumb_3_link_geom</geom>
-				<updateRate>100.0</updateRate>
-				<controller:gazebo_ros_bumper name="${name}_thumb_3_gazebo_ros_bumper_controller" plugin="libgazebo_ros_bumper.so">
+			<sensor name='${name}_thumb_3_contact_sensor' type='contact'>
+				<always_on>true</always_on>
+				<update_rate>100</update_rate>
+				<contact>
+					<collision>${name}_thumb_3_link_geom</collision>
+				</contact>
+				<plugin name="${name}_thumb_3_gazebo_ros_bumper_controller" filename="libgazebo_ros_bumper.so">
 					<alwaysOn>true</alwaysOn>
 					<updateRate>100.0</updateRate>
 					<frameName>${name}_thumb_3_link</frameName>
 					<bumperTopicName>${name}_thumb_3_bumper</bumperTopicName>
-					<interface:bumper name="${name}_thumb_3_bumper_iface" />
-				</controller:gazebo_ros_bumper>
-			</sensor:contact>
-			<material>IPA/Grey2</material>
+				</plugin>
+			</sensor>
+			<material>Schunk/LightGrey</material>
 		</gazebo>
 	</xacro:macro>

File: schunk_description/urdf/sdh/sdh.urdf.xacro (robot description, xacro)
@@ -24,5 +24,5 @@
 					<mesh filename="package://schunk_description/meshes/sdh/palm.stl" />
 				</geometry>
-				<material name="IPA/DarkGrey" />
+				<material name="Schunk/LightGrey" />
 			</visual>
 			<collision>
@@ -68,5 +68,5 @@
 					<mesh filename="package://schunk_description/meshes/sdh/knuckle.stl" />
 				</geometry>
-				<material name="IPA/Black" />
+				<material name="Schunk/LightGrey" />
 			</visual>
 			<collision>
@@ -97,5 +97,5 @@
 					<mesh filename="package://schunk_description/meshes/sdh/finger.stl" />
 				</geometry>
-			<material name="IPA/DarkGrey" />
+			<material name="Schunk/LightGrey" />
 			</visual>
 			<collision>
@@ -126,5 +126,5 @@
 					<mesh filename="package://schunk_description/meshes/sdh/finger_tip.stl" />
 				</geometry>
-				<material name="IPA/Black" />
+				<material name="Schunk/LightGrey" />
 			</visual>
 			<collision>
@@ -157,5 +157,5 @@
 					<mesh filename="package://schunk_description/meshes/sdh/knuckle.stl" />
 				</geometry>
-				<material name="IPA/Black" />
+				<material name="Schunk/LightGrey" />
 			</visual>
 			<collision>
@@ -186,5 +186,5 @@
 					<mesh filename="package://schunk_description/meshes/sdh/finger.stl" />
 				</geometry>
-				<material name="IPA/DarkGrey" />
+				<material name="Schunk/LightGrey" />
 			</visual>
 			<collision>
@@ -215,5 +215,5 @@
 					<mesh filename="package://schunk_description/meshes/sdh/finger_tip.stl" />
 				</geometry>
-				<material name="IPA/Black" />
+				<material name="Schunk/LightGrey" />
 			</visual>
 			<collision>
@@ -242,5 +242,5 @@
 					<mesh filename="package://schunk_description/meshes/sdh/knuckle.stl" />
 				</geometry>
-				<material name="IPA/Black" />
+				<material name="Schunk/LightGrey" />
 			</visual>
 			<collision>
@@ -271,5 +271,5 @@
 					<mesh filename="package://schunk_description/meshes/sdh/finger.stl" />
 				</geometry>
-				<material name="IPA/DarkGrey" />
+				<material name="Schunk/LightGrey" />
 			</visual>
 			<collision>
@@ -300,5 +300,5 @@
 					<mesh filename="package://schunk_description/meshes/sdh/finger_tip.stl" />
 				</geometry>
-				<material name="IPA/Black" />
+				<material name="Schunk/LightGrey" />
 			</visual>
 			<collision>
