Commit message: workable ipython control changes in urdf's : now using dae not stl there is also working shadow copy of hand

File: schunk_description/urdf/sdh/sdh.urdf.xacro (robot description, xacro)
@@ -22,12 +22,12 @@
 				<origin xyz="0 0 0" rpy="0 0 0" />
 				<geometry>
-					<mesh filename="package://schunk_description/meshes/sdh/palm.stl" />
-				</geometry>
-				<material name="Schunk/LightGrey" />
-			</visual>
-			<collision>
-				<origin xyz="0 0 0" rpy="0 0 0" />
-				<geometry>
-					<mesh filename="package://schunk_description/meshes/sdh/palm.stl"/>
+					<mesh filename="package://schunk_description/meshes/sdh/palm.dae" />
+				</geometry>
+				<material name="Schunk/LightGrey" />
+			</visual>
+			<collision>
+				<origin xyz="0 0 0" rpy="0 0 0" />
+				<geometry>
+					<mesh filename="package://schunk_description/meshes/sdh/palm.dae"/>
 				</geometry>
 			</collision>
@@ -66,12 +66,12 @@
 				<origin xyz="0 0 0" rpy="0 0 0" />
 				<geometry>
-					<mesh filename="package://schunk_description/meshes/sdh/knuckle.stl" />
-				</geometry>
-				<material name="Schunk/LightGrey" />
-			</visual>
-			<collision>
-				<origin xyz="0 0 0" rpy="0 0 0" />
-				<geometry>
-				<mesh filename="package://schunk_description/meshes/sdh/knuckle.stl"/>
+					<mesh filename="package://schunk_description/meshes/sdh/knuckle.dae" />
+				</geometry>
+				<material name="Schunk/LightGrey" />
+			</visual>
+			<collision>
+				<origin xyz="0 0 0" rpy="0 0 0" />
+				<geometry>
+				<mesh filename="package://schunk_description/meshes/sdh/knuckle.dae"/>
 				</geometry>
 			</collision>
@@ -95,5 +95,5 @@
 				<origin xyz="0 0 0" rpy="0 0 0" />
 				<geometry>
-					<mesh filename="package://schunk_description/meshes/sdh/finger.stl" />
+					<mesh filename="package://schunk_description/meshes/sdh/finger.dae" />
 				</geometry>
 			<material name="Schunk/LightGrey" />
@@ -102,5 +102,5 @@
 				<origin xyz="0 0 0" rpy="0 0 0" />
 				<geometry>
-					<mesh filename="package://schunk_description/meshes/sdh/finger.stl"/>
+					<mesh filename="package://schunk_description/meshes/sdh/finger.dae"/>
 				</geometry>
 			</collision>
@@ -124,12 +124,12 @@
 				<origin xyz="0 0 0" rpy="0 0 0" />
 				<geometry>
-					<mesh filename="package://schunk_description/meshes/sdh/finger_tip.stl" />
-				</geometry>
-				<material name="Schunk/LightGrey" />
-			</visual>
-			<collision>
-				<origin xyz="0 0 0" rpy="0 0 0" />
-				<geometry>
-					<mesh filename="package://schunk_description/meshes/sdh/finger_tip.stl"/>
+					<mesh filename="package://schunk_description/meshes/sdh/finger_tip.dae" />
+				</geometry>
+				<material name="Schunk/LightGrey" />
+			</visual>
+			<collision>
+				<origin xyz="0 0 0" rpy="0 0 0" />
+				<geometry>
+					<mesh filename="package://schunk_description/meshes/sdh/finger_tip.dae"/>
 				</geometry>
 			</collision>
@@ -155,12 +155,12 @@
 				<origin xyz="0 0 0" rpy="0 0 0" />
 				<geometry>
-					<mesh filename="package://schunk_description/meshes/sdh/knuckle.stl" />
-				</geometry>
-				<material name="Schunk/LightGrey" />
-			</visual>
-			<collision>
-				<origin xyz="0 0 0" rpy="0 0 0" />
-				<geometry>
-					<mesh filename="package://schunk_description/meshes/sdh/knuckle.stl"/>
+					<mesh filename="package://schunk_description/meshes/sdh/knuckle.dae" />
+				</geometry>
+				<material name="Schunk/LightGrey" />
+			</visual>
+			<collision>
+				<origin xyz="0 0 0" rpy="0 0 0" />
+				<geometry>
+					<mesh filename="package://schunk_description/meshes/sdh/knuckle.dae"/>
 				</geometry>
 			</collision>
@@ -184,12 +184,12 @@
 				<origin xyz="0 0 0" rpy="0 0 0" />
 				<geometry>
-					<mesh filename="package://schunk_description/meshes/sdh/finger.stl" />
-				</geometry>
-				<material name="Schunk/LightGrey" />
-			</visual>
-			<collision>
-				<origin xyz="0 0 0" rpy="0 0 0" />
-				<geometry>
-					<mesh filename="package://schunk_description/meshes/sdh/finger.stl"/>
+					<mesh filename="package://schunk_description/meshes/sdh/finger.dae" />
+				</geometry>
+				<material name="Schunk/LightGrey" />
+			</visual>
+			<collision>
+				<origin xyz="0 0 0" rpy="0 0 0" />
+				<geometry>
+					<mesh filename="package://schunk_description/meshes/sdh/finger.dae"/>
 				</geometry>
 			</collision>
@@ -213,12 +213,12 @@
 				<origin xyz="0 0 0" rpy="0 0 0" />
 				<geometry>
-					<mesh filename="package://schunk_description/meshes/sdh/finger_tip.stl" />
-				</geometry>
-				<material name="Schunk/LightGrey" />
-			</visual>
-			<collision>
-				<origin xyz="0 0 0" rpy="0 0 0" />
-				<geometry>
-					<mesh filename="package://schunk_description/meshes/sdh/finger_tip.stl"/>
+					<mesh filename="package://schunk_description/meshes/sdh/finger_tip.dae" />
+				</geometry>
+				<material name="Schunk/LightGrey" />
+			</visual>
+			<collision>
+				<origin xyz="0 0 0" rpy="0 0 0" />
+				<geometry>
+					<mesh filename="package://schunk_description/meshes/sdh/finger_tip.dae"/>
 				</geometry>
 			</collision>
@@ -240,12 +240,12 @@
 				<origin xyz="0 0 0" rpy="0 0 0" />
 				<geometry>
-					<mesh filename="package://schunk_description/meshes/sdh/knuckle.stl" />
-				</geometry>
-				<material name="Schunk/LightGrey" />
-			</visual>
-			<collision>
-				<origin xyz="0 0 0" rpy="0 0 0" />
-				<geometry>
-					<mesh filename="package://schunk_description/meshes/sdh/knuckle.stl"/>
+					<mesh filename="package://schunk_description/meshes/sdh/knuckle.dae" />
+				</geometry>
+				<material name="Schunk/LightGrey" />
+			</visual>
+			<collision>
+				<origin xyz="0 0 0" rpy="0 0 0" />
+				<geometry>
+					<mesh filename="package://schunk_description/meshes/sdh/knuckle.dae"/>
 				</geometry>
 			</collision>
@@ -269,12 +269,12 @@
 				<origin xyz="0 0 0" rpy="0 0 0" />
 				<geometry>
-					<mesh filename="package://schunk_description/meshes/sdh/finger.stl" />
-				</geometry>
-				<material name="Schunk/LightGrey" />
-			</visual>
-			<collision>
-				<origin xyz="0 0 0" rpy="0 0 0" />
-				<geometry>
-					<mesh filename="package://schunk_description/meshes/sdh/finger.stl"/>
+					<mesh filename="package://schunk_description/meshes/sdh/finger.dae" />
+				</geometry>
+				<material name="Schunk/LightGrey" />
+			</visual>
+			<collision>
+				<origin xyz="0 0 0" rpy="0 0 0" />
+				<geometry>
+					<mesh filename="package://schunk_description/meshes/sdh/finger.dae"/>
 				</geometry>
 			</collision>
@@ -298,12 +298,12 @@
 				<origin xyz="0 0 0" rpy="0 0 0" />
 				<geometry>
-					<mesh filename="package://schunk_description/meshes/sdh/finger_tip.stl" />
-				</geometry>
-				<material name="Schunk/LightGrey" />
-			</visual>
-			<collision>
-				<origin xyz="0 0 0" rpy="0 0 0" />
-				<geometry>
-					<mesh filename="package://schunk_description/meshes/sdh/finger_tip.stl"/>
+					<mesh filename="package://schunk_description/meshes/sdh/finger_tip.dae" />
+				</geometry>
+				<material name="Schunk/LightGrey" />
+			</visual>
+			<collision>
+				<origin xyz="0 0 0" rpy="0 0 0" />
+				<geometry>
+					<mesh filename="package://schunk_description/meshes/sdh/finger_tip.dae"/>
 				</geometry>
 			</collision>
